Commit message: minor fixes
- steering angle lookup table function fixed
- urdf model changed
- footprint changed
- added launch parameters

File: src/simulation/data/urdf_model/apollo_13.urdf (robot description, URDF)
Before this commit: robot blinky, 14 links, 13 joints
Links:
- link base_footprint: geometry visual box size=.40 .20 0
- link base_link: geometry visual box size=.40 .20 .18
