Commit message: dynamic reconfigure + fixes

File: src/apollo_13/data/urdf_model/apollo_13.urdf (robot description, URDF)
Before this commit: robot blinky, 9 links, 8 joints
Links:
- added link base_laser; visual box size=.066 .24 .066
- added link front_sensor; visual box size=.05 .05 .05
- added link left_sensor; visual box size=.05 .05 .05
- added link right_sensor; visual box size=.05 .05 .05
- added link scan; visual box size=0 0 0
- link base_footprint: geometry visual box size=.40 .20 0
- link base_link: geometry visual box size=.40 .20 .18
Joints:
- added joint base_laser_joint: type fixed, parent base_link, child base_laser, origin xyz=.18 0 .1
- added joint front_sensor_joint: type fixed, parent base_link, child front_sensor, origin xyz=.175 0 -.06
- added joint left_sensor_joint: type fixed, parent base_link, child left_sensor, origin xyz=0 .1 -.06 rpy=0 0 1.57
- added joint right_sensor_joint: type fixed, parent base_link, child right_sensor, origin xyz=0 -.1 -.06 rpy=0 0 -1.57
- added joint scan_joint: type fixed, parent base_laser, child scan, origin xyz=0 0 0
